Commit message: added force plugin

File: server/src/arm-model/urdf/arm.xacro (robot description, xacro)
@@ -82,7 +82,41 @@
               radius="0.15" length="0.25" />
   <!-- END - Robot description -->
-  <gazebo>
-    <plugin name="gazebo_ros_control" filename="libgazebo_ros_control.so">
-    </plugin>
+    <!-- This plugin will publish the joint_states for the selected joints
+            (which robot_state_publisher can then use to broadcast the approprate tf). -->
+    <gazebo>
+        <plugin name="gazebo_ros_joint_state_publisher"
+            filename="libgazebo_ros_joint_state_publisher.so">
+            <update_rate>20</update_rate>
+            <joint_name>"${link_00_name}"</joint_name>
+            <joint_name>link_01</joint_name>
+            <joint_name>link_02</joint_name>
+            <joint_name>link_03</joint_name>
+            <joint_name>link_05</joint_name>
+            <joint_name>link_06</joint_name>
+        </plugin>
+    </gazebo>
+    <!-- This plugin will read a JointTrajectory message from the /set_joint_trajectory topic
+            and move the machine accordingly. It's a bit clunky but it works. -->
+    <!-- You'll probably want to add damping to the joints to stop them it flopping around.
+            e.g. <dynamics damping="10.0" friction="10.0"/> -->
+    <!-- Here's an example message to publish to test it:
+            ros2 topic pub -1 /set_joint_trajectory trajectory_msgs/msg/JointTrajectory  '{header: {frame_id: world}, joint_names: [slider_joint, arm_joint], points: [  {positions: {0.8,0.6}} ]}' -->
+    <gazebo>
+        <plugin name="gazebo_ros_joint_pose_trajectory"
+            filename="libgazebo_ros_joint_pose_trajectory.so">
+            <update_rate>2</update_rate>
+        </plugin>
+    </gazebo>
+  <!-- Ros Gazebo force Plugin -->
+  <!-- http://wiki.ros.org/pr2_gazebo_plugins/Tutorials/Attaching%20a%20GazeboRosForce%20pugin%20to%20Objects%20in%20Simulation
+  ros2 pub /force geometry_msgs/Wrench  '{force:  {x: 0.0, y: 0.0, z: 0.0}, torque: {x: 0.0,y: 0.0,z: 0.6}}' -->
+   <gazebo>
+    <controller:gazebo_ros_force name="gazebo_ros_force" plugin="libgazebo_ros_force.so">
+      <alwaysOn>true</alwaysOn>
+      <update>100</update>
+      <updateRate>100.0</updateRate>
+      <bodyName>link_01</bodyName>
+      <topicName>force</topicName>
+    </controller:gazebo_ros_force>
   </gazebo>
 </robot>

File: server/src/arm-model/urdf/links_joints.xacro (robot description, xacro)
@@ -8,6 +8,7 @@
       <parent link="${parent}" />
       <child link="${child}" />
+      <dynamics damping="10.0" friction="10.0"/>
     </joint>
-    <transmission name="trans_${name}">
+    <!-- <transmission name="trans_${name}">
       <type>transmission_interface/SimpleTransmission</type>
       <joint name="${name}">
@@ -18,5 +19,5 @@
         <mechanicalReduction>1</mechanicalReduction>
       </actuator>
-    </transmission>
+    </transmission> -->
   </xacro:macro>
   <xacro:macro name="m_link_cylinder" params="name origin_xyz origin_rpy radius length mass ixx ixy ixz iyy iyz izz">
