Commit message: added more stuff

File: server/install/arm_model/share/arm_model/urdf/links_joints.xacro (robot description, xacro)
@@ -78,5 +78,5 @@
           <mesh filename="${meshfile}" scale="${meshscale}"/>
         </geometry>
-        <material name="light_black"/>
+        <!-- <material name="light_black"/> -->
       </visual>
     </link>
