Commit message: switched to ROS1

File: server-ros1/src/arm-model/urdf/arm.urdf (robot description, URDF)
Before this commit: robot mrm, 8 links, 7 joints
Links:
- removed link link_05
- added link ir_ranger, mass 0.1; collision box size=0.03 0.03 0.005; visual box size=0.03 0.03 0.005
- link link_clawL: geometry collision mesh filename=package://arm-model/meshes/gripperLeft.stl scale=0.001 0.001 0.001; visual mesh filename=package://arm-model/meshes/gripperLeft.stl scale=0.001 0.001 0.001
- link link_clawR: geometry collision mesh filename=package://arm-model/meshes/gripperRight.stl scale=0.001 0.001 0.001; visual mesh filename=package://arm-model/meshes/gripperRight.stl scale=0.001 0.001 0.001
Joints:
- removed joint link_04__link_05
- removed joint link_05__link_clawL
- removed joint link_05__link_clawR
- added joint ir_ranger__link_clawL: type revolute, parent ir_ranger, child link_clawL, origin xyz=0.03 -0.014  -0.00 rpy=0 0 0, axis 0 0 -1, limit lower=-0.6 upper=0.9 effort=1000 velocity=0.5
- added joint ir_ranger__link_clawR: type revolute, parent ir_ranger, child link_clawR, origin xyz=0.03 +0.014  -0.00 rpy=0 0 0, axis 0 0 1, limit lower=-0.6 upper=0.9 effort=1000 velocity=0.5
- added joint link_04__ir_ranger: type fixed, parent link_04, child ir_ranger, origin xyz=0.055 0 0 rpy=0 0 0
- joint base_link__link_01: axis 0 0 1 -> 0 0 -1
- joint link_01__link_02: limit lower=0.0 upper=1.5708 effort=1000 velocity=0.5 -> lower=-0.7854 upper=0.7854 effort=1000 velocity=0.5; origin xyz=0 0 0.029 rpy=0 0 0 -> xyz=0 0 0.029 rpy=0 -0.698 0
- joint link_02__link_03: axis 0 1 0 -> 0 -1 0; origin xyz=0.103 0 0.015 rpy=0 0 0 -> xyz=0.103 0 0.015 rpy=0 0.5584 0
- joint link_03__link_04: axis 0 1 0 -> 0 -1 0; origin xyz=0.065 0 -0.015 rpy=0 0 0 -> xyz=0.065 0 -0.015 rpy=0 1.047 0

File: server-ros1/src/arm-model/urdf/arm.xacro (robot description, xacro)
@@ -60,5 +60,5 @@
       iyy="0.1" iyz="0"
       izz="0.1"
-      meshfile="package://arm_model/meshes/gripperRight.stl"
+      meshfile="package://arm-model/meshes/gripperRight.stl"
       meshscale="0.001 0.001 0.001"
   />
@@ -69,5 +69,5 @@
       iyy="0.1" iyz="0"
       izz="0.1"
-      meshfile="package://arm_model/meshes/gripperLeft.stl"
+      meshfile="package://arm-model/meshes/gripperLeft.stl"
       meshscale="0.001 0.001 0.001"
   />
